File: a2k6c.kicad_pcb (KiCad board)
At the start: 2 copper layers, 41.3 x 43.8 mm, 12 parts, among them J1 Slot, J2 I^{2}C, J3 Buttons, U2 74LVC244, U3 74AHCT595, U4 74LVC244, U5 74AHCT1GU04

Commit message: ready to order first prototype.
Parts:
- added G1: Crankery, a2k6c:crankery_small, B.Cu at (45.8, 56.1)
- C1, C2, C3, C4, J2: moved to B.Cu
- U2, U4: moved to F.Cu
- ∏1: footprint a2k6c:MODULE_RP2040-ZERO -> a2k6c:MODULE_RP2040-ZERO_Basic
- moved C2 32.2 mm to (28.2, 47.1), turned to 90 degrees
- moved U5 30.9 mm to (29.6, 47.7)
- moved U3 28.4 mm to (32.1, 37.3)
- moved C1 27.9 mm to (33.0, 32.9)
- moved C3 18.5 mm to (59.1, 47.7), turned to -90 degrees
- moved U2 17.3 mm to (54.4, 51.9), turned to 0 degrees
- moved C4 13.8 mm to (44.9, 47.7), turned to -90 degrees
- moved U4 13.4 mm to (40.2, 51.9), turned to 0 degrees
- moved ∏1 6.97 mm to (51.6, 34.9), turned to -90 degrees
- moved J2 4.54 mm to (28.4, 28.1), turned to 0 degrees
- moved J3 2.08 mm to (30.2, 26.3), turned to 0 degrees
Routing:
- net Net-(J1-D2): track 0.00 -> 55.7 mm, vias 0 -> 2
- net Net-(J1-D3): track 0.00 -> 54.3 mm, vias 0 -> 1
- net Net-(J1-D1): track 0.00 -> 54.2 mm, vias 0 -> 2
- net Net-(J1-D4): track 0.00 -> 54.1 mm, vias 0 -> 1
- net /A_{0}: track 59.1 -> 8.79 mm, vias 3 -> 2
- net Net-(J1-D5): track 0.00 -> 50.1 mm, vias 0 -> 5
- net Net-(J1-D0): track 0.00 -> 47.5 mm, vias 0 -> 2
- net Net-(J1-D6): track 0.00 -> 43.7 mm, vias 0 -> 5
- net Net-(J1-D7): track 0.00 -> 41.8 mm, vias 0 -> 5
- net /A_{3}: track 53.8 -> 16.4 mm, vias 4 -> 0
- net /A_{2}: track 49.4 -> 12.8 mm, vias 3 -> 0
- net /A_{1}: track 45.5 -> 10.4 mm, vias 3 -> 0
- net Net-(J1-A12): track 0.00 -> 33.1 mm, vias 0 -> 3
- net /A_{4}: track 38.1 -> 7.81 mm, vias 3 -> 2
- net /A_{11}: track 0.00 -> 27.5 mm, vias 0 -> 2
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Other:
- board text added: "1"
- board text added: "2026-08-31 dave hamilton"
- board text added: "3.3V"
- board text added: "A2K6C"
- board text added: "r1"
- board text removed: "+3.3V"
- board text removed: "•1•"
