File: a2k6c.kicad_sch (KiCad schematic)
At the start: 12 parts, among them J1 Slot, J2 I^{2}C, J3 Buttons, U2 74LVC244, U3 74AHCT595, U4 74LVC244, U5 74AHCT1GU04

Commit message: ready to order first prototype.
Parts:
- added G1: Crankery, a2k6c:crankery_small, symbol a2k6c:crankery
- ∏1: footprint a2k6c:MODULE_RP2040-ZERO -> a2k6c:MODULE_RP2040-ZERO_Basic; symbol a2k6c:RP2040-ZERO -> a2k6c:RP2040-ZERO_Basic
Connections:
- net GND: no longer ∏1.33 (GND)
- no-connect marks 13 -> 4
Other:
- company: (none) -> Dave Hamilton
- title: (none) -> a2k6c
Changed lines of the file:
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@@
 	(generator_version "10.0")
 	(paper "A4")
+	(title_block
+		(title "a2k6c")
+		(date "2026-08-31")
+		(rev "rev 1")
+		(company "Dave Hamilton")
+	)
 	(junction
 		(at 62.23 60.96)
@@
 	)
 	(junction
-		(at 191.77 83.82)
-		(diameter 0)
-		(color 0 0 0 0)
-	)
-	(junction
 		(at 85.09 152.4)
 		(diameter 0)
@@
 	)
 	(no_connect
-		(at 212.09 40.64)
-	)
-	(no_connect
-		(at 212.09 35.56)
-	)
-	(no_connect
-		(at 212.09 38.1)
-	)
-	(no_connect
-		(at 212.09 45.72)
-	)
-	(no_connect
 		(at 62.23 110.49)
 	)
@@
 	)
 	(no_connect
-		(at 212.09 30.48)
-	)
-	(no_connect
-		(at 212.09 27.94)
-	)
-	(no_connect
-		(at 212.09 43.18)
-	)
-	(no_connect
-		(at 212.09 48.26)
-	)
-	(no_connect
 		(at 133.35 58.42)
 	)
@@
 		(at 62.23 107.95)
 	)
-	(no_connect
-		(at 212.09 33.02)
-	)
 	(wire
 		(pts
@@
 	(wire
 		(pts
-			(xy 191.77 83.82) (xy 196.85 83.82)
-		)
-		(stroke
-			(width 0)
-			(type default)
-		)
-	)
-	(wire
-		(pts
 			(xy 62.23 48.26) (xy 82.55 48.26)
 		)
@@
 	(symbol
 		(lib_id "power:GND")
-		(at 191.77 83.82 0)
+		(at 194.31 83.82 0)
 		(mirror y)
 		(unit 1)
@@
 		(fields_autoplaced yes)
 		(property "Reference" "#PWR08"
-			(at 191.77 90.17 0)
+			(at 194.31 90.17 0)
 			(hide yes)
 			(show_name no)
@@
 		)
 		(property "Value" "GND"
-			(at 191.77 88.9 0)
+			(at 194.31 88.9 0)
 			(show_name no)
 			(do_not_autoplace no)
@@
 		)
 		(property "Footprint" ""
-			(at 191.77 83.82 0)
+			(at 194.31 83.82 0)
 			(hide yes)
 			(show_name no)
@@
 		)
 		(property "Datasheet" ""
-			(at 191.77 83.82 0)
+			(at 194.31 83.82 0)
 			(hide yes)
 			(show_name no)
@@
 		)
 		(property "Description" "Power symbol creates a global label with name \"GND\" , ground"
-			(at 191.77 83.82 0)
+			(at 194.31 83.82 0)
 			(hide yes)
 			(show_name no)
@@
 	)
 	(symbol
-		(lib_id "a2k6c:RP2040-ZERO")
+		(lib_id "a2k6c:RP2040-ZERO_Basic")
 		(at 194.31 45.72 0)
 		(unit 1)
@@
 			)
 		)
-		(property "Footprint" "a2k6c:MODULE_RP2040-ZERO"
+		(property "Footprint" "a2k6c:MODULE_RP2040-ZERO_Basic"
 			(at 194.31 88.138 0)
 			(hide yes)
@@
 		(pin "13"
 		)
-		(pin "32"
-		)
 		(pin "7"
 		)
@@
 		(pin "1"
 		)
-		(pin "33"
-		)
-		(pin "24"
-		)
 		(pin "21"
 		)
-		(pin "29"
-		)
-		(pin "26"
-		)
-		(pin "30"
-		)
-		(pin "27"
-		)
-		(pin "25"
-		)
-		(pin "31"
-		)
-		(pin "28"
-		)
 		(instances
 			(project "a2k6c"
@@
 					(unit 1)
 				)
+			)
+		)
+	)
+	(symbol
+		(lib_id "a2k6c:crankery")
+		(at 30.48 175.26 0)
+		(unit 1)
+		(body_style 1)
+		(exclude_from_sim no)
+		(in_bom yes)
+		(on_board yes)
+		(in_pos_files yes)
+		(dnp no)
+		(fields_autoplaced yes)
+		(property "Reference" "G1"
+			(at 33.02 175.2599 0)
+			(show_name no)
+			(do_not_autoplace no)
+			(effects
+				(font
+					(size 1.27 1.27)
+				)
+				(justify left)
+			)
+		)
+		(property "Value" "Crankery"
+			(at 33.02 177.7999 0)
+			(show_name no)
+			(do_not_autoplace no)
+			(effects
+				(font
+					(size 1.27 1.27)
+				)
+				(justify left)
+			)
+		)
+		(property "Footprint" "a2k6c:crankery_small"
+			(at 30.48 175.26 0)
+			(hide yes)
+			(show_name no)
+			(do_not_autoplace no)
+			(effects
+				(font
+					(size 1.27 1.27)
+				)
+			)
+		)
+		(property "Datasheet" ""
+			(at 30.48 175.26 0)
+			(hide yes)
+			(show_name no)
+			(do_not_autoplace no)
+			(effects
+				(font
+					(size 1.27 1.27)
+				)
+			)
+		)
+		(property "Description" ""
+			(at 30.48 175.26 0)
+			(hide yes)
+			(show_name no)
+			(do_not_autoplace no)
+			(effects
+				(font
+					(size 1.27 1.27)
+				)
+			)
+		)
+		(instances
+			(project "a2k6c"
+				(path "/98178a74-9081-4441-88fc-ad854177256d"
+					(reference "G1")
+					(unit 1)
+				)
